File: gate_drive.kicad_sch (KiCad schematic)
At the start: 0 parts

Commit message: S4: gate drive — 3x UCC27524 single stage, hardware enable, DB37 frozen
Replaces 3.0's three-stage chain ('1G126 x6 -> CD4504B -> AND gate powered
from GPIO131) with one stage: 3x UCC27524 dual 5A drivers whose input and
enable thresholds are fixed and independent of VDD, so 3.3V logic switches a
13.5V output stage directly.

The PrimeSTACK datasheet (user-supplied mid-session, now in datasheets/) is
the authoritative source for the DB37 and overturned five inherited beliefs:
  - fault is HIGH, not LOW  -> hw_control_v2.h MODULE_FAULT_ACTIVE_LOW is
    inverted; also makes a disconnected DB37 read as FAULT (fail-safe)
  - analog outputs drive 5 mA -> S5 needs no Vbus buffer op-amp
  - one NTC pin (29), and it is the 10 V channel -> NTC_2_* retired
  - pins 9/27 are a 15V/50mA supply OUTPUT; 3.0 shorted pin 27 to GND
  - pin 1 is true earth/shield, not GND
Bench items #1, #2 and #4 are answered on paper; #5 halves.

Topology chosen on availability first, per the roadmap rule: the whole
TC446x/MIC446x quad family is dead at JLC (TC4468: 14 in stock) against
9550 for the UCC27524.

Safety fix caught during capture: the F28379D powers up with GPIO pull-ups
enabled, so 100k pull-downs would have left the enable and PWM inputs near
2.7V — all six gates armed while the MCU is in reset. Pull-downs are 4.7k.
The enable net's pull-down is 1k because six UCC27524 EN pins present 33k of
internal pull-up to 13.5V.

Numbers: module sees 12.95-13.62 V against an 11-15 V window (validating the
13.5 V rail from S3); worst-case skew 53 ns = 3.5% of the 1500 ns deadband;
effective deadtime 1399 ns; gate path draws ~10 mA.

ARCH CHANGES: NTC_2_RAW/NTC_2_ADC retired; SW_MAIN_3V3 now also feeds
gate_drive as the interlock term; new global net PGND_MOD (DB37 10/28) tied
to GND only at NT2, the 24 V entry star.

gate_drive: 56 components, 44 nets, ERC 0 violations on the sheet, netlist
verified node-by-node (44/44). Libraries 46/46 symbols, 40/40 footprints.
Every part carries an LCSC fiel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
Parts:
- added C29, C31, C33: 1uF 50V, FE_UFPR_4_0:C_0805_2012Metric, symbol FE_UFPR_4_0:C
- added C30, C32, C34, C35: 100nF 50V, FE_UFPR_4_0:C_0603_1608Metric, symbol FE_UFPR_4_0:C
- added C36: 10uF 50V, FE_UFPR_4_0:C_1206_3216Metric, symbol FE_UFPR_4_0:C
- added C37, C38, C39, C40, C41, C42, C43: 1nF C0G, FE_UFPR_4_0:C_0603_1608Metric, symbol FE_UFPR_4_0:C
- added D9: RED GATE_EN, FE_UFPR_4_0:LED_0603_1608Metric, symbol FE_UFPR_4_0:LED
- added J2: DSUB-37_Socket, FE_UFPR_4_0:DSUB-37_Socket_Horizontal_P2.77x2.54mm_MountingHoles, symbol FE_UFPR_4_0:DSUB-37_Socket
- added JP1: ILOCK_SEL, FE_UFPR_4_0:SolderJumper-3_P1.3mm_Open_Pad1.0x1.5mm_NumberLabels, symbol FE_UFPR_4_0:SolderJumper_3_Open
- added JP2: SHLD_TIE, FE_UFPR_4_0:SolderJumper-2_P1.3mm_Open_Pad1.0x1.5mm, symbol FE_UFPR_4_0:SolderJumper_2_Open
- added R18, R19, R20, R21, R22, R23: 100R, FE_UFPR_4_0:R_0603_1608Metric, symbol FE_UFPR_4_0:R
- added R24, R25, R26, R27, R28, R29: 10k, FE_UFPR_4_0:R_0603_1608Metric, symbol FE_UFPR_4_0:R
- added R30, R31, R32, R36, R37, R38, R39, R40, R41: 4.7k, FE_UFPR_4_0:R_0603_1608Metric, symbol FE_UFPR_4_0:R
- added R33: 1k, FE_UFPR_4_0:R_0603_1608Metric, symbol FE_UFPR_4_0:R
- added R34: 680R, FE_UFPR_4_0:R_0603_1608Metric, symbol FE_UFPR_4_0:R
- added R35: 1M, FE_UFPR_4_0:R_0603_1608Metric, symbol FE_UFPR_4_0:R
- added TP10: TP_PWM_UH, FE_UFPR_4_0:TestPoint_Pad_D1.5mm, symbol FE_UFPR_4_0:TestPoint
- added TP11: TP_PWM_UL, FE_UFPR_4_0:TestPoint_Pad_D1.5mm, symbol FE_UFPR_4_0:TestPoint
- added TP12: TP_PWM_VH, FE_UFPR_4_0:TestPoint_Pad_D1.5mm, symbol FE_UFPR_4_0:TestPoint
- added TP13: TP_PWM_VL, FE_UFPR_4_0:TestPoint_Pad_D1.5mm, symbol FE_UFPR_4_0:TestPoint
- added TP14: TP_PWM_WH, FE_UFPR_4_0:TestPoint_Pad_D1.5mm, symbol FE_UFPR_4_0:TestPoint
- added TP15: TP_PWM_WL, FE_UFPR_4_0:TestPoint_Pad_D1.5mm, symbol FE_UFPR_4_0:TestPoint
- added TP16: TP_GATE_EN, FE_UFPR_4_0:TestPoint_Pad_D1.5mm, symbol FE_UFPR_4_0:TestPoint
- added TP17: TP_MOD15V_1, FE_UFPR_4_0:TestPoint_Pad_D1.5mm, symbol FE_UFPR_4_0:TestPoint
- added TP18: TP_MOD15V_2, FE_UFPR_4_0:TestPoint_Pad_D1.5mm, symbol FE_UFPR_4_0:TestPoint
- added U5, U6, U7: UCC27524DR, FE_UFPR_4_0:SOIC-8_3.9x4.9mm_P1.27mm, symbol FE_UFPR_4_0:UCC27524D
- added U8: SN74LVC1G11DBVR, FE_UFPR_4_0:SOT-23-6, symbol FE_UFPR_4_0:74LVC1G11
Connections:
- net DRV_EN_3V3: now also R30.1, U8.1
- net DRV_EN_AUX_3V3: now also R31.1, U8.3
- net FLT_OC_A_15V: now also J2.2
- net FLT_OC_B_15V: now also J2.22
- net FLT_OC_C_15V: now also J2.5
- net FLT_OT_15V: now also J2.6
- net FLT_OV_15V: now also J2.16
- net ISNS_A_RAW: now also J2.30
- net ISNS_B_RAW: now also J2.31
- net ISNS_C_RAW: now also J2.32
- net ISNS_RTN: now also J2.12, J2.13
- net NTC_1_RAW: now also J2.29
- net PWM_UH_3V3: now also R36.1, U5.2 (INA)
- net PWM_UL_3V3: now also R37.1, U5.4 (INB)
- net PWM_VH_3V3: now also R38.1, U6.2 (INA)
- net PWM_VL_3V3: now also R39.1, U6.4 (INB)
- net PWM_WH_3V3: now also R40.1, U7.2 (INA)
- net PWM_WL_3V3: now also R41.1, U7.4 (INB)
- net VBUS_RTN: now also J2.11
- net VBUS_SNS_RAW: now also J2.7
- new net +13V5_GATE: C29.1, C30.1, C31.1, C32.1, C33.1, C34.1, C36.1, U5.6 (V_{DD}), U6.6 (V_{DD}), U7.6 (V_{DD})
- new net +24V_MOD: J2.26, J2.8
- new net +3V3: C35.1, JP1.3 (B), U8.5 (VCC)
- new net GATE_EN_3V3: R33.1, R34.1, TP16.1, U5.1 (ENA), U5.8 (ENB), U6.1 (ENA), U6.8 (ENB), U7.1 (ENA), U7.8 (ENB), U8.4
- new net GATE_ILOCK_3V3: JP1.2 (C), R32.1, U8.6
- new net GND: C29.2, C30.2, C31.2, C32.2, C33.2, C34.2, C35.2, C36.2, C37.2, C38.2, C39.2, C40.2, C41.2, C42.2, C43.2, D9.1 (K), J2.19, J2.25, J2.37, JP2.2 (B), R24.2, R25.2, R26.2, R27.2, R28.2, R29.2, R30.2, R31.2, R32.2, R33.2, R35.2, R36.2, R37.2, R38.2, R39.2, R40.2, R41.2, U5.3 (GND), U6.3 (GND), U7.3 (GND), U8.2 (GND)
- new net LED_GATE_EN: D9.2 (A), R34.2
- new net MOD_AUX15V_1: J2.9, TP17.1
- new net MOD_AUX15V_2: J2.27, TP18.1
- new net PGND_MOD: J2.10, J2.28
- new net PWM_UH_15V: C37.1, J2.21, R18.2, R24.1, TP10.1
- new net PWM_UH_DRV: R18.1, U5.7 (OUTA)
- new net PWM_UL_15V: C38.1, J2.20, R19.2, R25.1, TP11.1
- new net PWM_UL_DRV: R19.1, U5.5 (OUTB)
- new net PWM_VH_15V: C39.1, J2.4, R20.2, R26.1, TP12.1
- new net PWM_VH_DRV: R20.1, U6.7 (OUTA)
- new net PWM_VL_15V: C40.1, J2.3, R21.2, R27.1, TP13.1
- new net PWM_VL_DRV: R21.1, U6.5 (OUTB)
- new net PWM_WH_15V: C41.1, J2.24, R22.2, R28.1, TP14.1
- new net PWM_WH_DRV: R22.1, U7.7 (OUTA)
- new net PWM_WL_15V: C42.1, J2.23, R23.2, R29.1, TP15.1
- new net PWM_WL_DRV: R23.1, U7.5 (OUTB)
- new net SHIELD_DB37: C43.1, J2.1, J2.G1 (SHIELD), J2.G2 (SHIELD), JP2.1 (A), R35.1
- new net SW_MAIN_3V3: JP1.1 (A)
- no-connect marks 0 -> 8
Other:
- note added: "DB37 PIN TABLE - from Infineon-6PS04512E43W39693-DS-v02_00 p.6 (circuit diagram) Module connector is SUB-D 37 male, UNC4/40 female thread. Board side = socket. 1 True earth / shield SHIELD_DB37 20 HB A IGBT BOT PWM_UL_15V 2 HB A error FLT_OC_A_15V 21 HB A IGBT TOP PWM_UH_15V 3 HB B IGBT BOT PWM_VL_15V 22 HB B error FLT_OC_B_15V 4 HB B IGBT TOP PWM_VH_15V 23 HB C IGBT BOT PWM_WL_15V 5 HB C error F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"
- note added: "DC LEVELS AT THE MODULE INPUT (datasheet p.2: input network = 10k to GND + 1nF to GND) R24-R29 (10k) + C37-C42 (1nF C0G) fit that network on our side; if the module also has it, R = 5k. Rail 13.500V +/-2% = 13.23..13.77V. Driver ROH 5R (8.5R max) + R_series 100R. V(module) = 13.23 x 5000/5105 = 12.96V worst case min ... 13.63V max. Window is 11-15V. => margin >= 1.96V below the 11V minimum and >=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"
- note added: "FAIL-SAFE TABLE - every case lands GATES OFF LaunchPad unplugged PWM 4k7 || 120k internal to GND; U8 inputs 4k7 to GND -> EN LOW MCU in reset F28379D GPIO pull-ups are ENABLED at reset (worst case ~24k): PWM node = 3.3 x 4.52k/28.5k = 0.52V and U8 in = 0.54V, both < 0.8V VIL. OK +3V3 dead, +13V5 alive U8 out high-Z (Ioff); R33 1k beats 6x 200k EN pull-ups -> EN 0.39V (0.76V worst). OK Board dead,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"
- note added: "JP1 INTERLOCK SELECT (default 1-2 = interlock ACTIVE) JP2 SHIELD TIE (default open = soft RC tie) 1-2 GATE_EN gated by SW_MAIN_3V3 from vehicle_io <-- DEFAULT open DB37 shell + pin 1 'true earth/shield' 2-3 interlock bypassed to +3V3 (BENCH ONLY) tied to GND via C43 1nF || R35 1M Exclusive 3-pad jumper: the two sources can never fight. closed hard tie to GND (per S2 shield policy)"
- note added: "POLARITY CHAIN - ACTIVE HIGH END TO END (matches hw_control_v2.h) GPIO6 HIGH -> PWM_UH_3V3 HIGH -> U5.INA (non-inverting, VIH 2.3V max, threshold independent of VDD) -> U5.OUTA HIGH ~13.5V -> R18 100R -> DB37 pin 21 'HB A IGBT TOP' >= 11V = module logic HIGH = ON Datasheet p.2: 'Digital input level ... logic high = on'. U/V/W = module half-bridge A/B/C. ENABLE: GATE_EN_3V3 = DRV_EN(GPIO66) AND DR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"
- note added: "S10 LAYOUT NOTES (gate drive) 1. C29/C31/C33 (1uF) and C30/C32/C34 (100nF) within 2mm of each UCC27524 VDD/GND; VDD loop area minimal. 2. R18-R23 immediately at the driver outputs, NOT at the connector - they damp the harness at the source. 3. R24-R29 + C37-C42 at the DB37 pins (far end of the board trace), per the datasheet input network. 4. Route the six gate lines as one grouped bus of equal l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"
- note added: "S4 - GATE DRIVE 3V3 -> 13.5V single stage, hardware enable gating, DB37 to PrimeSTACK 3x UCC27524 (dual 5A, TTL inputs independent of VDD, per-channel ENABLE) replace 3.0's 6x '1G126 + CD4504B + GPIO-powered AND. All values from Infineon-6PS04512E43W39693-DS-v02_00 (datasheets/) - see S4_GATE_DRIVE_DESIGN.md for every derivation."
- note added: "SKEW vs 1500 ns DEADBAND (PWM_DEADBAND_NS in hw_control_v2.h) UCC27524: tD1/tD2 = 17ns typ / 27ns max; in-package channel matching 1ns typ / 2ns max; tR 6/10ns, tF 10/14ns. R 1% and C0G 5% => RC spread +/-5%, identical on all six channels. RC at the module pin: (100R + 5R) x (1nF ours + 1nF module + ~0.1nF cable) = 220ns. rise to 11V = -tau*ln(1-11/13.37) = 380ns fall to 1.5V = tau*ln(13.37/1.5) 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"
