File: gate_drive.kicad_sch (KiCad schematic)
At the start: 56 parts, among them J2 DSUB-37_Socket, U5 UCC27524DR, U6 UCC27524DR, U7 UCC27524DR, U8 SN74LVC1G11DBVR

Commit message: More routing
Connections:
- net PWM_UH_15V: now also R19.2; no longer R18.2
- net PWM_UH_3V3: now also R37.1, U5.4 (INB); no longer R36.1, U5.2 (INA)
- net PWM_UH_DRV: now also R19.1, U5.5 (OUTB); no longer R18.1, U5.7 (OUTA)
- net PWM_UL_15V: now also R18.2; no longer R19.2
- net PWM_UL_3V3: now also R36.1, U5.2 (INA); no longer R37.1, U5.4 (INB)
- net PWM_UL_DRV: now also R18.1, U5.7 (OUTA); no longer R19.1, U5.5 (OUTB)
- net PWM_VH_15V: now also R21.2; no longer R20.2
- net PWM_VH_3V3: now also R39.1, U6.4 (INB); no longer R38.1, U6.2 (INA)
- net PWM_VH_DRV: now also R21.1, U6.5 (OUTB); no longer R20.1, U6.7 (OUTA)
- net PWM_VL_15V: now also R20.2; no longer R21.2
- net PWM_VL_3V3: now also R38.1, U6.2 (INA); no longer R39.1, U6.4 (INB)
- net PWM_VL_DRV: now also R20.1, U6.7 (OUTA); no longer R21.1, U6.5 (OUTB)
- net PWM_WH_15V: now also R23.2; no longer R22.2
- net PWM_WH_3V3: now also R41.1, U7.4 (INB); no longer R40.1, U7.2 (INA)
- net PWM_WH_DRV: now also R23.1, U7.5 (OUTB); no longer R22.1, U7.7 (OUTA)
- net PWM_WL_15V: now also R22.2; no longer R23.2
- net PWM_WL_3V3: now also R40.1, U7.2 (INA); no longer R41.1, U7.4 (INB)
- net PWM_WL_DRV: now also R22.1, U7.7 (OUTA); no longer R23.1, U7.5 (OUTB)
Other:
- note added: "POLARITY CHAIN - ACTIVE HIGH END TO END (matches hw_control_v2.h) GPIO6 HIGH -> PWM_UH_3V3 HIGH -> U5.INB (non-inverting, VIH 2.3V max, threshold independent of VDD) -> U5.OUTB HIGH ~13.5V -> R19 100R -> DB37 pin 21 'HB A IGBT TOP' >= 11V = module logic HIGH = ON Datasheet p.2: 'Digital input level ... logic high = on'. U/V/W = module half-bridge A/B/C. ENABLE: GATE_EN_3V3 = DRV_EN(GPIO66) AND DR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"
- note removed: "POLARITY CHAIN - ACTIVE HIGH END TO END (matches hw_control_v2.h) GPIO6 HIGH -> PWM_UH_3V3 HIGH -> U5.INA (non-inverting, VIH 2.3V max, threshold independent of VDD) -> U5.OUTA HIGH ~13.5V -> R18 100R -> DB37 pin 21 'HB A IGBT TOP' >= 11V = module logic HIGH = ON Datasheet p.2: 'Digital input level ... logic high = on'. U/V/W = module half-bridge A/B/C. ENABLE: GATE_EN_3V3 = DRV_EN(GPIO66) AND DR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"
- moved on the sheet: C37, C38, C39, C40, C41, C42, R24, R25, R26, R27, R28, R29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
