File: gate_drive.kicad_sch (KiCad schematic)
At the start: 56 parts, among them J2 DSUB-37_Socket, U5 UCC27524DR, U6 UCC27524DR, U7 UCC27524DR, U8 SN74LVC1G11DBVR

Commit message: S12: fab package (fab/), C22936->C22935 fix, firmware handoff, CPL audit seed
- fix six 1 MOhm positions that carried C22936 (1 Ohm): R35 R67 R77 R89 R104 R118 -> C22935 in the sheets and on the board footprints (LCSC field only; ERC 0, DRC parity 0, netlist = golden.net)
- fab/: gerbers (11 layers + Excellon PTH/NPTH), JLC BOM (70 lines) + CPL (289 parts, board-corner origin, rotations 0-360), jlc_verify record, README with order options
- tools/fab: make_package.sh (rebuilds fab/), jlc_bomcpl.py (--origin, --hand-solder, prefix rotation table), jlc_verify.py (VALUE_MISMATCH check), jlc_rotations.json (community seed, unverified), fix_c22936.sh
- S12_FAB_PACKAGE.md (decisions D1-D6, CPL audit table, assembly notes, bring-up sheet, TP map), S12_FIRMWARE_HANDOFF.md (control_v2_pinmap.md answered line by line)
- decisions: U4 JLC-placed, Economic single-side + 12 B.Cu parts hand-soldered, HW_NAME FE_UFPR_4_0, no coating before bring-up
- DECISION_LOG, OPEN_ITEMS, JLC_PARTS (S12 re-verification), CLAUDE.md phase paragraph
- not yet orderable: CPL rotation offsets must be confirmed on JLC's placement preview before v4.0-release

Co-Authored-By: Claude Fable 5.1 <noreply@anthropic.com>
Claude-Session: https://claude.ai/code/session_01RJcYQJpnw6FjWqUDikqjUU
Parts:
- R35: LCSC C22936 -> C22935
Changed lines of the file:
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@@
 			)
 		)
-		(property "LCSC" "C22936"
+		(property "LCSC" "C22935"
 			(at 228.6 170.18 0)
 			(hide yes)
