File: power.kicad_sch (KiCad schematic)
At the start: 0 parts

Commit message: S3: power supplies — entry protection, 13.5V/5V/3V3 rails, isolated ±15V
power sheet captured: 79 components, 30 nets, ERC 0 violations on the sheet,
netlist verified node-by-node, 64 LCSC fields set, zero placeholder values.

Both converters named in the roadmap were rejected. LMR33630 and TPS62153 each
have no MODE pin, so neither can be forced out of light-load PFM — and on a board
that samples every analog channel at 10 kHz, a load-dependent burst rate is exactly
the wrong failure mode. Replacements:

  +13V5_GATE  TPS54360B  60 V (survives the 53.3 V SMBJ33A clamp; a 36 V part does
              not), 500 kHz, 47 uH sized to hold CCM down to 0.13 A, external
              compensation 5.6k/47nF/120pF, UVLO 15.37/13.26 V
  +5V         TPS62933F  FCCM — fixed 1.2 MHz at any load incl. LaunchPad unplugged,
              and the only family member without spread spectrum. This is the rail
              that feeds every analog front-end.

Three hardware-destroying traps caught during capture: TPS54360 EN is rated 8.4 V
max and TPS62933F EN 6.0 V max (neither may be tied to its input rail — both now
divided), and the TPS62933F SS pin cannot float (>=6.8 nF required).

Divider values were re-picked against live JLC stock, not E96 tables: the natural
162k/10.2k pair is unbuyable (1 and 3 units in stock), as is the exact 5.49k
compensation resistor (19). Final picks are Basic/high-stock parts.

Gate rail set to 13.566 V (user decision, S3/S4 joint) — centres the module in its
11-15 V HIGH window so S4 is free to pick any damping resistor <=100 ohm.

Two ARCH CHANGES: rail +12V_GATE renamed +13V5_GATE, and new global net +24V_MOD
for the fused (3 A) module-aux pass-through to DB37 8/26.

Library grown 28->41 symbols and 19->35 footprints. Two footprints derived because
KiCad ships neither: the Littelfuse 451 2410 fuse land (the only in-stock 5 A SMD
fuse with an adequate voltage rating) and the Mornsun URA2415YMD-6WR3 DIP module.

Also: .history/ (the MCP checkpoint repo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
Parts:
- added C1: 100uF 50V, FE_UFPR_4_0:CP_Elec_8x10.5, symbol FE_UFPR_4_0:C_Polarized
- added C10, C14, C2, C23, C3, C5, C9: 10uF 50V, FE_UFPR_4_0:C_1206_3216Metric, symbol FE_UFPR_4_0:C
- added C11, C12, C15, C19, C22, C24, C26, C28, C4, C8: 100nF 50V, FE_UFPR_4_0:C_0603_1608Metric, symbol FE_UFPR_4_0:C
- added C13, C6: 47nF 50V, FE_UFPR_4_0:C_0603_1608Metric, symbol FE_UFPR_4_0:C
- added C16, C17, C18, C20, C21, C25, C27: 10uF 25V, FE_UFPR_4_0:C_0805_2012Metric, symbol FE_UFPR_4_0:C
- added C7: 120pF C0G, FE_UFPR_4_0:C_0603_1608Metric, symbol FE_UFPR_4_0:C
- added D1: SMBJ33A, FE_UFPR_4_0:D_SMB, symbol FE_UFPR_4_0:D_TVS_Unidirectional
- added D2: BZX84C15, FE_UFPR_4_0:SOT-23, symbol FE_UFPR_4_0:D_Zener
- added D3: SS36, FE_UFPR_4_0:D_SMA, symbol FE_UFPR_4_0:D_Schottky
- added D4: red +24V_PROT, FE_UFPR_4_0:LED_0603_1608Metric, symbol FE_UFPR_4_0:LED
- added D5: red +13V5_GATE, FE_UFPR_4_0:LED_0603_1608Metric, symbol FE_UFPR_4_0:LED
- added D6: red +5V, FE_UFPR_4_0:LED_0603_1608Metric, symbol FE_UFPR_4_0:LED
- added D7: red +3V3, FE_UFPR_4_0:LED_0603_1608Metric, symbol FE_UFPR_4_0:LED
- added D8: red +15V_ISO, FE_UFPR_4_0:LED_0603_1608Metric, symbol FE_UFPR_4_0:LED
- added F1: 5A 125V, FE_UFPR_4_0:Fuse_2410_6125Metric, symbol FE_UFPR_4_0:Fuse
- added F2: 3A 63V, FE_UFPR_4_0:Fuse_1206_3216Metric, symbol FE_UFPR_4_0:Fuse
- added J1: Mini-Fit Jr 5566-02A, FE_UFPR_4_0:Molex_Mini-Fit_Jr_5566-02A_2x01_P4.20mm_Vertical, symbol FE_UFPR_4_0:Conn_01x02
- added L1: 47uH, FE_UFPR_4_0:L_Changjiang_FNR8040S, symbol FE_UFPR_4_0:L
- added L2: 3.3uH, FE_UFPR_4_0:L_Changjiang_FNR5040S, symbol FE_UFPR_4_0:L
- added NT1: ISO_COM-GND, FE_UFPR_4_0:NetTie-2_SMD_Pad0.5mm, symbol FE_UFPR_4_0:NetTie_2
- added Q1: SQD50P06-15L, FE_UFPR_4_0:TO-252-2, symbol FE_UFPR_4_0:MOSFET_P_GDS
- added R1, R8: 100k, FE_UFPR_4_0:R_0603_1608Metric, symbol FE_UFPR_4_0:R
- added R10: 52.3k, FE_UFPR_4_0:R_0603_1608Metric, symbol FE_UFPR_4_0:R
- added R11, R13: 10k, FE_UFPR_4_0:R_0603_1608Metric, symbol FE_UFPR_4_0:R
- added R12: 0R, FE_UFPR_4_0:R_0603_1608Metric, symbol FE_UFPR_4_0:R
- added R14, R6: 4.7k, FE_UFPR_4_0:R_0603_1608Metric, symbol FE_UFPR_4_0:R
- added R15: 1.5k, FE_UFPR_4_0:R_0603_1608Metric, symbol FE_UFPR_4_0:R
- added R16: 680R, FE_UFPR_4_0:R_0603_1608Metric, symbol FE_UFPR_4_0:R
- added R17: 6.8k, FE_UFPR_4_0:R_0603_1608Metric, symbol FE_UFPR_4_0:R
- added R2: 620k, FE_UFPR_4_0:R_0603_1608Metric, symbol FE_UFPR_4_0:R
- added R3: 49.9k, FE_UFPR_4_0:R_0603_1608Metric, symbol FE_UFPR_4_0:R
- added R4: 200k, FE_UFPR_4_0:R_0603_1608Metric, symbol FE_UFPR_4_0:R
- added R5: 75k, FE_UFPR_4_0:R_0603_1608Metric, symbol FE_UFPR_4_0:R
- added R7: 5.6k, FE_UFPR_4_0:R_0603_1608Metric, symbol FE_UFPR_4_0:R
- added R9: 33k, FE_UFPR_4_0:R_0603_1608Metric, symbol FE_UFPR_4_0:R
- added TP1: +24V_PROT, FE_UFPR_4_0:TestPoint_Pad_D1.5mm, symbol FE_UFPR_4_0:TestPoint
- added TP2: +13V5_GATE, FE_UFPR_4_0:TestPoint_Pad_D1.5mm, symbol FE_UFPR_4_0:TestPoint
- added TP3: +5V, FE_UFPR_4_0:TestPoint_Pad_D1.5mm, symbol FE_UFPR_4_0:TestPoint
- added TP4: +3V3, FE_UFPR_4_0:TestPoint_Pad_D1.5mm, symbol FE_UFPR_4_0:TestPoint
- added TP5: +24V_MOD, FE_UFPR_4_0:TestPoint_Pad_D1.5mm, symbol FE_UFPR_4_0:TestPoint
- added TP6: +15V_ISO, FE_UFPR_4_0:TestPoint_Pad_D1.5mm, symbol FE_UFPR_4_0:TestPoint
- added TP7: -15V_ISO, FE_UFPR_4_0:TestPoint_Pad_D1.5mm, symbol FE_UFPR_4_0:TestPoint
- added TP8: ISO_COM, FE_UFPR_4_0:TestPoint_Pad_D1.5mm, symbol FE_UFPR_4_0:TestPoint
- added TP9: GND, FE_UFPR_4_0:TestPoint_Pad_D1.5mm, symbol FE_UFPR_4_0:TestPoint
- added U1: TPS54360BDDAR, FE_UFPR_4_0:TI_SO-PowerPAD-8_ThermalVias, symbol FE_UFPR_4_0:TPS54360DDA
- added U2: TPS62933FDRLR, FE_UFPR_4_0:SOT-583-8, symbol FE_UFPR_4_0:TPS62933F
- added U3: AMS1117-3.3, FE_UFPR_4_0:SOT-223-3_TabPin2, symbol FE_UFPR_4_0:AMS1117-3.3
- added U4: URA2415YMD-6WR3, FE_UFPR_4_0:Converter_DCDC_Mornsun_URA-YMD-6WR3_THT, symbol FE_UFPR_4_0:Converter_DCDC_URA-YMD_Dual
Connections:
- new net +13V5_GATE: C10.1, C11.1, C14.1, C15.1, C9.1, L1.2, R14.1, R5.1, R8.1, TP2.1, U2.3 (VIN)
- new net +15V_ISO: C25.1, C26.1, R17.1, TP6.1, U4.3 (+Vo)
- new net +24V_IN: F1.1, J1.1 (Pin_1)
- new net +24V_MOD: C5.1, F2.2, TP5.1
- new net +24V_PROT: C1.1, C2.1, C23.1, C24.1, C3.1, C4.1, D1.1 (K), D2.1 (K), F2.1, Q1.3 (S), R13.1, R2.1, TP1.1, U1.2 (VIN), U4.2 (+Vin)
- new net +3V3: C21.1, C22.1, R16.1, TP4.1, U3.2 (VO)
- new net +5V: C16.1, C17.1, C18.1, C19.1, C20.1, L2.2, R10.1, R15.1, TP3.1, U3.3 (VI)
- new net -15V_ISO: C27.2, C28.2, TP7.1, U4.5 (-Vo)
- new net GND: C1.2, C10.2, C11.2, C13.2, C14.2, C15.2, C16.2, C17.2, C18.2, C19.2, C2.2, C20.2, C21.2, C22.2, C23.2, C24.2, C3.2, C4.2, C5.2, C6.2, C7.2, C9.2, D1.2 (A), D3.2 (A), D4.1 (K), D5.1 (K), D6.1 (K), D7.1 (K), J1.2 (Pin_2), NT1.2, R1.2, R11.2, R3.2, R4.2, R6.2, R9.2, TP9.1, U1.7 (GND), U1.9 (GNDPAD), U2.1 (RT), U2.4 (GND), U3.1 (GND), U4.1 (-Vin)
- new net ISO_COM: C25.2, C26.2, C27.1, C28.1, D8.1 (K), NT1.1, TP8.1, U4.4 (0V)
- new net PWR_24V_FUSED: F1.2, Q1.2 (D)
- new net PWR_LED_13V5: D5.2 (A), R14.2
- new net PWR_LED_15V: D8.2 (A), R17.2
- new net PWR_LED_24V: D4.2 (A), R13.2
- new net PWR_LED_3V3: D7.2 (A), R16.2
- new net PWR_LED_5V: D6.2 (A), R15.2
- new net PWR_QGATE: D2.2 (A), Q1.1 (G), R1.1
- new net PWR_U1_BOOT: C8.1, U1.1 (BOOT)
- new net PWR_U1_COMP: C7.1, R7.1, U1.6 (COMP)
- new net PWR_U1_COMPC: C6.1, R7.2
- new net PWR_U1_EN: R2.2, R3.1, U1.3 (EN)
- new net PWR_U1_FB: R5.2, R6.1, U1.5 (FB)
- new net PWR_U1_RT: R4.1, U1.4 (RT/CLK)
- new net PWR_U1_SW: C8.2, D3.1 (K), L1.1, U1.8 (SW)
- new net PWR_U2_BST: R12.1, U2.6 (BST)
- new net PWR_U2_BSTC: C12.1, R12.2
- new net PWR_U2_EN: R8.2, R9.1, U2.2 (EN)
- new net PWR_U2_FB: R10.2, R11.1, U2.8 (FB)
- new net PWR_U2_SS: C13.1, U2.7 (SS)
- new net PWR_U2_SW: C12.2, L2.1, U2.5 (SW)
Other:
- note added: "EN PIN RATINGS - BOTH DIVIDERS ARE MANDATORY, NOT OPTIONAL: U1 EN abs max = 8.4V. R2/R3 = 620k/49.9k -> UVLO start 15.37V, stop 13.26V (both below the 18V spec minimum, so the board runs across the whole 18-30V range and stops cleanly on brownout). EN sits at 2.23V with 30V in, and only 3.95V even during a 53V TVS clamp event. U2 EN abs max = 6.0V. R8/R9 = 100k/33k -> EN = 3.37V off the 13.57V ra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"
- note added: "Q1 REVERSE-POLARITY ORIENTATION (easy to get backwards): P-channel body diode conducts DRAIN -> SOURCE, therefore DRAIN = input side, SOURCE = load side. Normal polarity: body diode forward + gate pulled to GND by R1 => Vgs approx -24V => hard on. Reverse polarity: Vgs approx 0 => off, body diode blocks. D2 (BZX84C15) IS MANDATORY - unclamped Vgs would be -24..-30V against the +/-20V Vgs limit. R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"
- note added: "S3 - POWER SUPPLIES +24V_IN (18-30V) -> +13V5_GATE 13.566V -> +5V 4.984V -> +3V3 plus isolated +/-15V All component values computed - see S3_POWER_DESIGN.md for every derivation, datasheet equation and JLC stock check."
- note added: "SWITCHING-MODE NOTES - this board samples every analog channel at 10kHz and noise >5kHz aliases irrecoverably: U2 is the "F" variant = FCCM, fixed 1.2MHz at ANY load including LaunchPad-unplugged, and it is the only family member WITHOUT spread spectrum. Do NOT substitute a plain TPS62933 - the 5V rail feeds every analog front-end, and a load-dependent PFM burst rate would land in the sampled ban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"
- note added: "U1 TPS54360B - PCB LAYOUT NOTES FOR S10 (datasheet SLVSBB4G section 10.1): - Bypass VIN to GND with low-ESR X5R/X7R ceramic (C4) as close to the VIN pin as possible. - MINIMISE the loop area formed by C4, the VIN pin and the ANODE of catch diode D3. This is the hot loop - it carries the fast di/dt and is the dominant radiator. - Tie the GND pin directly to the PowerPAD under the IC; stitch the Po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"
- note added: "U2 TPS62933F - PCB LAYOUT NOTES FOR S10 (datasheet SLUSEA4D section 12.1): - The input-capacitor / power-ground loop is THE most critical feature: wide, short, minimum area. - Inductor L2, input caps (C14/C15) and output caps (C16-C19) all on the SAME layer as the IC. - C15 (100nF) as close as physically possible to the VIN and GND pins - key to EMI reduction. - Keep the SW trace short and wide t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"

Commit message: S3 fix: revert gate-rail buck to LMR33630; input range 18-26 V; TVS -> SMCJ26A
The 60 V TPS54360B swap was wrong and is reverted. It rested on the S2 assumption
"+24V_IN (vehicle LV, 18-30 V)" from ARCHITECTURE.md §1, which I inherited and never
confirmed. The actual LV rail max is <=26 V, which makes a 36 V part correct.

Reverting is also a net simplification: the LMR33630 is synchronous (no catch diode),
internally compensated (no R/C/C network) and fixed 400 kHz (no RT resistor) — five
fewer parts and better efficiency.

  FB divider recomputed for Vref = 1.000 V (not 0.8 V): 150k/12k -> exactly 13.500 V,
    both JLC Basic, >400k stock each
  UVLO now via the EN divider 100k/10k (both already in the S1 kit): ratio 11,
    V_EN-H 1.231 V -> rising 13.5 V, V_EN-HYS 100 mV -> falling 12.4 V
  L1 47uH -> 22uH (C15857) per TI's ripple rule using the device's 3 A rating (24.6%);
    the rail runs PWM above ~0.35 A and PFM below
  C_VCC 1uF added (LMR33630 has an internal LDO); PG pin gets a no-connect flag

What survives from the detour is a finding about the TVS, not the buck: SMBJ33A breaks
down at 36.7-40.6 V, which straddles the LMR33630's 38 V absolute max, so that S2 pair
was genuinely broken. Replaced with SMCJ26A — same 42.1 V clamp spec but at 35.6 A
instead of 14.3 A, so at a realistic surge it sits near 30-34 V, safely under 38 V.

The TPS62153 -> TPS62933F swap on the 5 V rail STANDS and is unchanged. That rail feeds
every analog front-end, TPS62153's power-save mode cannot be defeated, and the swap is
independent of input voltage (U2 runs off the regulated 13.5 V rail).

Lesson logged in CLAUDE.md: two justifications were stacked for one decision (PFM and
voltage headroom) when only one was load-bearing — and that one rested on an unverified
inherited assumption.

ARCH CHANGE: input range narrowed 18-30 V -> 18-26 V.

75 components, 29 nets, ERC 0 violations on the power sheet, netlist verified node by
node, 60 LCSC fields. Libraries 43 symbols / 38 foot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
Parts:
- removed C7: 120pF C0G, FE_UFPR_4_0:C_0603_1608Metric, symbol FE_UFPR_4_0:C
- removed D3: SS36, FE_UFPR_4_0:D_SMA, symbol FE_UFPR_4_0:D_Schottky
- removed R4: 200k, FE_UFPR_4_0:R_0603_1608Metric, symbol FE_UFPR_4_0:R
- removed R7: 5.6k, FE_UFPR_4_0:R_0603_1608Metric, symbol FE_UFPR_4_0:R
- removed U1: TPS54360BDDAR, FE_UFPR_4_0:TI_SO-PowerPAD-8_ThermalVias, symbol FE_UFPR_4_0:TPS54360DDA
- added U1: LMR33630ADDAR, FE_UFPR_4_0:Texas_HSOP-8-1EP_3.9x4.9mm_P1.27mm_ThermalVias, symbol FE_UFPR_4_0:LMR33630ADDA
- C6: value 47nF 50V -> 1uF 50V; LCSC C1622 -> C15849
- D1: value SMBJ33A -> SMCJ26A; footprint FE_UFPR_4_0:D_SMB -> FE_UFPR_4_0:D_SMC; LCSC C19077586 -> C310042
- L1: value 47uH -> 22uH; footprint FE_UFPR_4_0:L_Changjiang_FNR8040S -> FE_UFPR_4_0:L_Sunlord_SWPA8040S; LCSC C168137 -> C15857
- R2: value 620k -> 100k; LCSC C23219 -> C25803
- R3: value 49.9k -> 10k; LCSC C23184 -> C25804
- R5: value 75k -> 150k; LCSC C23242 -> C22807
- R6: value 4.7k -> 12k; LCSC C23162 -> C22790
Connections:
- net +24V_PROT: now also U1.2 (VIN)
- net GND: now also U1.1 (GND), U1.9 (GND)
- net PWR_U1_BOOT: now also U1.7 (BOOT)
- net PWR_U1_EN: now also U1.3 (EN)
- net PWR_U1_FB: now also U1.5 (FB)
- net PWR_U1_SW: now also U1.8 (SW)
- net PWR_U1_COMPC renamed PWR_U1_VCC
- net PWR_U1_VCC: now also U1.6 (VCC)
- no-connect marks 0 -> 1
Other:
- note added: "EN / UVLO: U1 LMR33630 EN may be tied to VIN (abs max = VIN + 0.3 V), but R2/R3 = 100k/10k give a PROGRAMMABLE UVLO instead: divider ratio 11, V_EN-H = 1.231 V -> rising 13.5 V, V_EN-HYS = 100 mV -> falling 12.4 V. Both thresholds sit below the 18 V minimum input, so the board runs over the whole 18-26 V range and shuts down cleanly on a brownout rather than sagging the gate rail below the module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"
- note added: "Q1 REVERSE-POLARITY ORIENTATION (easy to get backwards): P-channel body diode conducts DRAIN -> SOURCE, therefore DRAIN = input side, SOURCE = load side. Normal polarity: body diode forward + gate pulled to GND by R1 => Vgs approx -24V => hard on. Reverse polarity: Vgs approx 0 => off, body diode blocks. D2 (BZX84C15) IS MANDATORY - unclamped Vgs would be -24..-30V against the +/-20V Vgs limit. D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"
- note added: "S3 - POWER SUPPLIES +24V_IN (18-26V) -> +13V5_GATE 13.500V -> +5V 4.984V -> +3V3 plus isolated +/-15V All component values computed - see S3_POWER_DESIGN.md for every derivation, datasheet equation and JLC stock check."
- note added: "U1 LMR33630A - PCB LAYOUT NOTES FOR S10 (datasheet SNVSAN3F section 10.1): - The input-capacitor / power-ground loop is THE most critical feature: wide, short, minimum area. VIN and GND pins are adjacent on the SOIC package, which simplifies this. - Place C4 (input bypass) as close as possible to the VIN and GND pins. - Place C6 (VCC bypass, 1uF) close to the VCC pin, short and wide traces to VCC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"
- note removed: "EN PIN RATINGS - BOTH DIVIDERS ARE MANDATORY, NOT OPTIONAL: U1 EN abs max = 8.4V. R2/R3 = 620k/49.9k -> UVLO start 15.37V, stop 13.26V (both below the 18V spec minimum, so the board runs across the whole 18-30V range and stops cleanly on brownout). EN sits at 2.23V with 30V in, and only 3.95V even during a 53V TVS clamp event. U2 EN abs max = 6.0V. R8/R9 = 100k/33k -> EN = 3.37V off the 13.57V ra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"
- note removed: "Q1 REVERSE-POLARITY ORIENTATION (easy to get backwards): P-channel body diode conducts DRAIN -> SOURCE, therefore DRAIN = input side, SOURCE = load side. Normal polarity: body diode forward + gate pulled to GND by R1 => Vgs approx -24V => hard on. Reverse polarity: Vgs approx 0 => off, body diode blocks. D2 (BZX84C15) IS MANDATORY - unclamped Vgs would be -24..-30V against the +/-20V Vgs limit. R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"
- note removed: "S3 - POWER SUPPLIES +24V_IN (18-30V) -> +13V5_GATE 13.566V -> +5V 4.984V -> +3V3 plus isolated +/-15V All component values computed - see S3_POWER_DESIGN.md for every derivation, datasheet equation and JLC stock check."
- note removed: "U1 TPS54360B - PCB LAYOUT NOTES FOR S10 (datasheet SLVSBB4G section 10.1): - Bypass VIN to GND with low-ESR X5R/X7R ceramic (C4) as close to the VIN pin as possible. - MINIMISE the loop area formed by C4, the VIN pin and the ANODE of catch diode D3. This is the hot loop - it carries the fast di/dt and is the dominant radiator. - Tie the GND pin directly to the PowerPAD under the IC; stitch the Po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"

Commit message: S4: gate drive — 3x UCC27524 single stage, hardware enable, DB37 frozen
Replaces 3.0's three-stage chain ('1G126 x6 -> CD4504B -> AND gate powered
from GPIO131) with one stage: 3x UCC27524 dual 5A drivers whose input and
enable thresholds are fixed and independent of VDD, so 3.3V logic switches a
13.5V output stage directly.

The PrimeSTACK datasheet (user-supplied mid-session, now in datasheets/) is
the authoritative source for the DB37 and overturned five inherited beliefs:
  - fault is HIGH, not LOW  -> hw_control_v2.h MODULE_FAULT_ACTIVE_LOW is
    inverted; also makes a disconnected DB37 read as FAULT (fail-safe)
  - analog outputs drive 5 mA -> S5 needs no Vbus buffer op-amp
  - one NTC pin (29), and it is the 10 V channel -> NTC_2_* retired
  - pins 9/27 are a 15V/50mA supply OUTPUT; 3.0 shorted pin 27 to GND
  - pin 1 is true earth/shield, not GND
Bench items #1, #2 and #4 are answered on paper; #5 halves.

Topology chosen on availability first, per the roadmap rule: the whole
TC446x/MIC446x quad family is dead at JLC (TC4468: 14 in stock) against
9550 for the UCC27524.

Safety fix caught during capture: the F28379D powers up with GPIO pull-ups
enabled, so 100k pull-downs would have left the enable and PWM inputs near
2.7V — all six gates armed while the MCU is in reset. Pull-downs are 4.7k.
The enable net's pull-down is 1k because six UCC27524 EN pins present 33k of
internal pull-up to 13.5V.

Numbers: module sees 12.95-13.62 V against an 11-15 V window (validating the
13.5 V rail from S3); worst-case skew 53 ns = 3.5% of the 1500 ns deadband;
effective deadtime 1399 ns; gate path draws ~10 mA.

ARCH CHANGES: NTC_2_RAW/NTC_2_ADC retired; SW_MAIN_3V3 now also feeds
gate_drive as the interlock term; new global net PGND_MOD (DB37 10/28) tied
to GND only at NT2, the 24 V entry star.

gate_drive: 56 components, 44 nets, ERC 0 violations on the sheet, netlist
verified node-by-node (44/44). Libraries 46/46 symbols, 40/40 footprints.
Every part carries an LCSC fiel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
Parts:
- added NT2: PGND_MOD-GND star, FE_UFPR_4_0:NetTie-2_SMD_Pad0.5mm, symbol FE_UFPR_4_0:NetTie_2
- TP1, TP2, TP3, TP4, TP5, TP6, TP7, TP8, TP9: LCSC (none) -> NOFIT
Connections:
- net GND: now also NT2.2
- new net PGND_MOD: NT2.1
Changed lines of the file:
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@@
 			)
 		)
+      (property "LCSC" "NOFIT"
+        (at 0 0 0)
+        (effects
+          (font
+            (size 1.27 1.27)
+          )
+          (hide yes)
+        )
+      )
 		(property "Description" "test point"
 			(at 320.04 190.5 0)
@@
 			)
 		)
+      (property "LCSC" "NOFIT"
+        (at 0 0 0)
+        (effects
+          (font
+            (size 1.27 1.27)
+          )
+          (hide yes)
+        )
+      )
 		(property "Description" "test point"
 			(at 340.36 190.5 0)
@@
 			)
 		)
+      (property "LCSC" "NOFIT"
+        (at 0 0 0)
+        (effects
+          (font
+            (size 1.27 1.27)
+          )
+          (hide yes)
+        )
+      )
 		(property "Description" "test point"
 			(at 359.41 190.5 0)
@@
 			)
 		)
+      (property "LCSC" "NOFIT"
+        (at 0 0 0)
+        (effects
+          (font
+            (size 1.27 1.27)
+          )
+          (hide yes)
+        )
+      )
 		(property "Description" "test point"
 			(at 379.73 190.5 0)
@@
 			)
 		)
+      (property "LCSC" "NOFIT"
+        (at 0 0 0)
+        (effects
+          (font
+            (size 1.27 1.27)
+          )
+          (hide yes)
+        )
+      )
 		(property "Description" "test point"
 			(at 400.05 190.5 0)
@@
 			)
 		)
+      (property "LCSC" "NOFIT"
+        (at 0 0 0)
+        (effects
+          (font
+            (size 1.27 1.27)
+          )
+          (hide yes)
+        )
+      )
 		(property "Description" "test point"
 			(at 320.04 224.79 0)
@@
 			)
 		)
+      (property "LCSC" "NOFIT"
+        (at 0 0 0)
+        (effects
+          (font
+            (size 1.27 1.27)
+          )
+          (hide yes)
+        )
+      )
 		(property "Description" "test point"
 			(at 340.36 224.79 0)
@@
 			)
 		)
+      (property "LCSC" "NOFIT"
+        (at 0 0 0)
+        (effects
+          (font
+            (size 1.27 1.27)
+          )
+          (hide yes)
+        )
+      )
 		(property "Description" "test point"
 			(at 359.41 224.79 0)
@@
 			)
 		)
+      (property "LCSC" "NOFIT"
+        (at 0 0 0)
+        (effects
+          (font
+            (size 1.27 1.27)
+          )
+          (hide yes)
+        )
+      )
 		(property "Description" "test point"
 			(at 379.73 224.79 0)
@@
 		(at 165.1 67.31)
 	)
+	(symbol
+		(lib_id "FE_UFPR_4_0:NetTie_2")
+		(at 30.48 64.77 0)
+		(unit 1)
+		(body_style 1)
+		(exclude_from_sim no)
+		(in_bom yes)
+		(on_board yes)
+		(in_pos_files yes)
+		(dnp no)
+		(property "Reference" "NT2"
+			(at 30.48 62.23 0)
+			(show_name no)
+			(do_not_autoplace no)
+			(effects
+				(font
+					(size 1.27 1.27)
+				)
+			)
+		)
+		(property "Value" "PGND_MOD-GND star"
+			(at 30.48 67.31 0)
+			(show_name no)
+			(do_not_autoplace no)
+			(effects
+				(font
+					(size 1.27 1.27)
+				)
+			)
+		)
+		(property "Footprint" "FE_UFPR_4_0:NetTie-2_SMD_Pad0.5mm"
+			(at 30.48 64.77 0)
+			(hide yes)
+			(show_name no)
+			(do_not_autoplace no)
+			(effects
+				(font
+					(size 1.27 1.27)
+				)
+			)
+		)
+		(property "Datasheet" ""
+			(at 30.48 64.77 0)
+			(hide yes)
+			(show_name no)
+			(do_not_autoplace no)
+			(effects
+				(font
+					(size 1.27 1.27)
+				)
+			)
+		)
+      (property "LCSC" "NOFIT"
+        (at 0 0 0)
+        (effects
+          (font
+            (size 1.27 1.27)
+          )
+          (hide yes)
+        )
+      )
+		(property "Description" "Net tie, 2 pins"
+			(at 30.48 64.77 0)
+			(hide yes)
+			(show_name no)
+			(do_not_autoplace no)
+			(effects
+				(font
+					(size 1.27 1.27)
+				)
+			)
+		)
+		(pin "1"
+		)
+		(pin "2"
+		)
+		(instances
+			(project "FE_UFPR_4_0"
+				(path "/f36b3dbb-4842-44d3-ae27-d77d669e5268"
+					(reference "NT2")
+					(unit 1)
+				)
+				(path "/0cde0ae3-e31e-4592-8212-8a072a248a80/6442f421-491d-4bfb-bee7-d0b4e843a827"
+					(reference "NT2")
+					(unit 1)
+				)
+			)
+		)
+	)
+	(global_label "PGND_MOD"
+		(at 27.94 64.77 180)
+		(effects
+			(font
+				(size 1.27 1.27)
+			)
+			(justify right)
+		)
+	)
+	(global_label "GND"
+		(at 33.02 64.77 0)
+		(effects
+			(font
+				(size 1.27 1.27)
+			)
+			(justify left)
+		)
+	)
 	(sheet_instances
