File: power.kicad_sch (KiCad schematic)
At the start: 70 parts, among them J1 Mini-Fit Jr 5566-02A, Q1 SQD50P06-15L, U1 LMR33630ADDAR, U2 TPS62933FDRLR, U3 AMS1117-3.3, U4 URA2415YMD-6WR3

Commit message: Placing rest blocks
Changed lines of the file:
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@@
 		)
 		(property "Value" "URA2415YMD-6WR3"
-			(at 245.11 147.32 0)
+			(at 245.11 141.478 0)
 			(show_name no)
 			(do_not_autoplace no)

Commit message: More routing
Parts:
- D2: symbol FE_UFPR_4_0:D_Zener -> FE_UFPR_4_0:D_Zener_SOT-23
Connections:
- net +24V_PROT: now also D2.3 (K); no longer D2.1 (K)
- net PWR_QGATE: now also D2.1 (A); no longer D2.2 (A)
Changed lines of the file:
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@@
 	)
 	(symbol
-		(lib_id "FE_UFPR_4_0:D_Zener")
+		(lib_id "FE_UFPR_4_0:D_Zener_SOT-23")
 		(at 78.74 44.45 270)
 		(unit 1)
@@
 			)
 		)
+		(pin "3"
+		)
 		(pin "1"
 		)
-		(pin "2"
-		)
 		(instances
