File: power.kicad_sch (KiCad schematic)
At the start: 70 parts, among them J1 Mini-Fit Jr 5566-02A, Q1 SQD50P06-15L, U1 LMR33630ADDAR, U2 TPS62933FDRLR, U3 AMS1117-3.3, U4 URA2415YMD-6WR3

Commit message: ROuting power planes
Connections:
- net +24V_MOD: now also C23.1, C24.1
- net +24V_PROT: no longer C23.1, C24.1
- net GND: no longer C23.2, C24.2, U4.1 (-Vin)
- net PGND_MOD: now also C23.2, C24.2, U4.1 (-Vin)
Other:
- moved on the sheet: C23, C24
Changed lines of the file:
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@@
 	)
 	(junction
+		(at 208.28 165.1)
+		(diameter 0)
+		(color 0 0 0 0)
+	)
+	(junction
+		(at 208.28 154.94)
+		(diameter 0)
+		(color 0 0 0 0)
+	)
+	(junction
+		(at 73.66 83.82)
+		(diameter 0)
+		(color 0 0 0 0)
+	)
+	(junction
 		(at 186.69 58.42)
 		(diameter 0)
@@
 	(wire
 		(pts
-			(xy 33.02 110.49) (xy 40.64 110.49)
-		)
-		(stroke
-			(width 0)
-			(type default)
-		)
-	)
-	(wire
-		(pts
 			(xy 275.59 125.73) (xy 287.02 125.73)
 		)
@@
 	(wire
 		(pts
+			(xy 208.28 163.83) (xy 208.28 165.1)
+		)
+		(stroke
+			(width 0)
+			(type default)
+		)
+	)
+	(wire
+		(pts
 			(xy 224.79 63.5) (xy 224.79 66.04)
 		)
@@
 	(wire
 		(pts
+			(xy 223.52 156.21) (xy 223.52 154.94)
+		)
+		(stroke
+			(width 0)
+			(type default)
+		)
+	)
+	(wire
+		(pts
 			(xy 40.64 93.98) (xy 46.99 93.98)
 		)
@@
 	(wire
 		(pts
-			(xy 20.32 110.49) (xy 27.94 110.49)
+			(xy 26.67 110.49) (xy 27.94 110.49)
 		)
 		(stroke
@@
 	(wire
 		(pts
-			(xy 198.12 58.42) (xy 214.63 58.42)
+			(xy 208.28 154.94) (xy 204.47 154.94)
 		)
 		(stroke
@@
 	(wire
 		(pts
-			(xy 78.74 40.64) (xy 91.44 40.64)
+			(xy 198.12 58.42) (xy 214.63 58.42)
 		)
 		(stroke
@@
 	(wire
 		(pts
-			(xy 257.81 135.89) (xy 275.59 135.89)
+			(xy 78.74 40.64) (xy 91.44 40.64)
 		)
 		(stroke
@@
 	(wire
 		(pts
-			(xy 257.81 125.73) (xy 275.59 125.73)
+			(xy 257.81 135.89) (xy 275.59 135.89)
 		)
 		(stroke
@@
 	(wire
 		(pts
-			(xy 224.79 52.07) (xy 224.79 55.88)
+			(xy 257.81 125.73) (xy 275.59 125.73)
 		)
 		(stroke
@@
 	(wire
 		(pts
-			(xy 232.41 125.73) (xy 219.71 125.73)
+			(xy 224.79 52.07) (xy 224.79 55.88)
 		)
 		(stroke
@@
 	(wire
 		(pts
-			(xy 68.58 165.1) (xy 68.58 167.64)
+			(xy 232.41 125.73) (xy 219.71 125.73)
 		)
 		(stroke
@@
 	(wire
 		(pts
-			(xy 88.9 76.2) (xy 104.14 76.2)
+			(xy 68.58 165.1) (xy 68.58 167.64)
 		)
 		(stroke
@@
 	(wire
 		(pts
-			(xy 20.32 93.98) (xy 33.02 93.98)
+			(xy 26.67 93.98) (xy 33.02 93.98)
 		)
 		(stroke
@@
 	(wire
 		(pts
-			(xy 73.66 76.2) (xy 88.9 76.2)
-		)
-		(stroke
-			(width 0)
-			(type default)
-		)
-	)
-	(wire
-		(pts
 			(xy 160.02 71.12) (xy 160.02 76.2)
 		)
@@
 	(wire
 		(pts
-			(xy 73.66 83.82) (xy 88.9 83.82)
-		)
-		(stroke
-			(width 0)
-			(type default)
-		)
-	)
-	(wire
-		(pts
 			(xy 196.85 71.12) (xy 196.85 68.58)
 		)
@@
 	(wire
 		(pts
+			(xy 223.52 163.83) (xy 223.52 165.1)
+		)
+		(stroke
+			(width 0)
+			(type default)
+		)
+	)
+	(wire
+		(pts
+			(xy 33.02 110.49) (xy 53.34 110.49)
+		)
+		(stroke
+			(width 0)
+			(type default)
+		)
+	)
+	(wire
+		(pts
 			(xy 243.84 93.98) (xy 256.54 93.98)
 		)
@@
 	(wire
 		(pts
+			(xy 223.52 154.94) (xy 208.28 154.94)
+		)
+		(stroke
+			(width 0)
+			(type default)
+		)
+	)
+	(wire
+		(pts
 			(xy 287.02 86.36) (xy 287.02 88.9)
 		)
@@
 	(wire
 		(pts
+			(xy 208.28 156.21) (xy 208.28 154.94)
+		)
+		(stroke
+			(width 0)
+			(type default)
+		)
+	)
+	(wire
+		(pts
+			(xy 208.28 165.1) (xy 204.47 165.1)
+		)
+		(stroke
+			(width 0)
+			(type default)
+		)
+	)
+	(wire
+		(pts
 			(xy 170.18 55.88) (xy 180.34 55.88)
 		)
@@
 	(wire
 		(pts
-			(xy 88.9 83.82) (xy 104.14 83.82)
+			(xy 73.66 83.82) (xy 78.74 83.82)
 		)
 		(stroke
@@
 	(wire
 		(pts
+			(xy 223.52 165.1) (xy 208.28 165.1)
+		)
+		(stroke
+			(width 0)
+			(type default)
+		)
+	)
+	(wire
+		(pts
 			(xy 281.94 166.37) (xy 294.64 166.37)
 		)
@@
 		)
 	)
-	(global_label "GND"
+	(global_label "PGND_MOD"
 		(shape bidirectional)
 		(at 219.71 135.89 180)
@@
 	(global_label "GND"
 		(shape bidirectional)
-		(at 104.14 83.82 270)
+		(at 78.74 83.82 270)
 		(effects
 			(font
@@
 		)
 		(property "Intersheetrefs" "${INTERSHEET_REFS}"
-			(at 104.14 83.82 0)
+			(at 78.74 83.82 0)
 			(hide yes)
 			(show_name no)
@@
 	(global_label "+24V_PROT"
 		(shape bidirectional)
-		(at 20.32 93.98 0)
+		(at 26.67 93.98 180)
 		(effects
 			(font
 				(size 1.27 1.27)
 			)
-			(justify left)
+			(justify right)
 		)
 		(property "Intersheetrefs" "${INTERSHEET_REFS}"
-			(at 20.32 93.98 0)
+			(at 26.67 93.98 0)
+			(hide yes)
+			(show_name no)
+			(do_not_autoplace no)
+			(effects
+				(font
+					(size 1.27 1.27)
+				)
+			)
+		)
+	)
+	(global_label "PGND_MOD"
+		(shape bidirectional)
+		(at 204.47 165.1 180)
+		(effects
+			(font
+				(size 1.27 1.27)
+			)
+			(justify right)
+		)
+		(property "Intersheetrefs" "${INTERSHEET_REFS}"
+			(at 204.47 165.1 0)
 			(hide yes)
 			(show_name no)
@@
 	(global_label "GND"
 		(shape bidirectional)
-		(at 40.64 110.49 270)
+		(at 53.34 110.49 270)
 		(effects
 			(font
@@
 		)
 		(property "Intersheetrefs" "${INTERSHEET_REFS}"
-			(at 40.64 110.49 0)
+			(at 53.34 110.49 0)
 			(hide yes)
 			(show_name no)
@@
 		)
 	)
+	(global_label "+24V_MOD"
+		(shape bidirectional)
+		(at 204.47 154.94 180)
+		(effects
+			(font
+				(size 1.27 1.27)
+			)
+			(justify right)
+		)
+		(property "Intersheetrefs" "${INTERSHEET_REFS}"
+			(at 204.47 154.94 0)
+			(hide yes)
+			(show_name no)
+			(do_not_autoplace no)
+			(effects
+				(font
+					(size 1.27 1.27)
+				)
+			)
+		)
+	)
 	(global_label "GND"
 		(shape bidirectional)
@@
 	(global_label "PGND_MOD"
 		(shape bidirectional)
-		(at 20.32 110.49 0)
+		(at 26.67 110.49 180)
 		(effects
 			(font
 				(size 1.27 1.27)
 			)
-			(justify left)
+			(justify right)
 		)
 		(property "Intersheetrefs" "${INTERSHEET_REFS}"
-			(at 20.32 110.49 0)
+			(at 26.67 110.49 0)
 			(hide yes)
 			(show_name no)
@@
 		)
 		(property "Value" "PGND_MOD-GND star"
-			(at 30.48 114.935 0)
+			(at 43.18 114.935 0)
 			(show_name no)
 			(do_not_autoplace no)
@@
 	(symbol
 		(lib_id "FE_UFPR_4_0:C")
-		(at 88.9 80.01 0)
+		(at 208.28 160.02 0)
 		(unit 1)
 		(body_style 1)
@@
 		(dnp no)
 		(property "Reference" "C23"
-			(at 92.202 78.74 0)
+			(at 211.582 158.75 0)
 			(show_name no)
 			(do_not_autoplace no)
@@
 		)
 		(property "Value" "10uF 50V"
-			(at 92.202 81.915 0)
+			(at 211.582 161.925 0)
 			(show_name no)
 			(do_not_autoplace no)
@@
 		)
 		(property "Footprint" "FE_UFPR_4_0:C_1206_3216Metric"
-			(at 88.9 80.01 0)
+			(at 208.28 160.02 0)
 			(hide yes)
 			(show_name no)
@@
 		)
 		(property "Datasheet" ""
-			(at 88.9 80.01 0)
+			(at 208.28 160.02 0)
 			(hide yes)
 			(show_name no)
@@
 		)
 		(property "Description" "Unpolarized capacitor"
-			(at 88.9 80.01 0)
+			(at 208.28 160.02 0)
 			(hide yes)
 			(show_name no)
@@
 		)
 		(property "LCSC" "C13585"
-			(at 88.9 80.01 0)
+			(at 208.28 160.02 0)
 			(hide yes)
 			(show_name no)
@@
 	(symbol
 		(lib_id "FE_UFPR_4_0:C")
-		(at 104.14 80.01 0)
+		(at 223.52 160.02 0)
 		(unit 1)
 		(body_style 1)
@@
 		(dnp no)
 		(property "Reference" "C24"
-			(at 107.442 78.74 0)
+			(at 226.822 158.75 0)
 			(show_name no)
 			(do_not_autoplace no)
@@
 		)
 		(property "Value" "100nF 50V"
-			(at 107.442 81.915 0)
+			(at 226.822 161.925 0)
 			(show_name no)
 			(do_not_autoplace no)
@@
 		)
 		(property "Footprint" "FE_UFPR_4_0:C_0603_1608Metric"
-			(at 104.14 80.01 0)
+			(at 223.52 160.02 0)
 			(hide yes)
 			(show_name no)
@@
 		)
 		(property "Datasheet" ""
-			(at 104.14 80.01 0)
+			(at 223.52 160.02 0)
 			(hide yes)
 			(show_name no)
@@
 		)
 		(property "Description" "Unpolarized capacitor"
-			(at 104.14 80.01 0)
+			(at 223.52 160.02 0)
 			(hide yes)
 			(show_name no)
@@
 		)
 		(property "LCSC" "C14663"
-			(at 104.14 80.01 0)
+			(at 223.52 160.02 0)
 			(hide yes)
 			(show_name no)
@@
 		)
 		(property "Value" "100nF 50V"
-			(at 76.962 81.915 0)
+			(at 76.708 80.264 0)
 			(show_name no)
 			(do_not_autoplace no)

Commit message: Silk fixes
Changed lines of the file:
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@@
+		)
+	)
+	(symbol
+		(lib_id "FE_UFPR_4_0:PWR_FLAG")
+		(at 26.67 110.49 180)
+		(unit 1)
+		(body_style 1)
+		(exclude_from_sim no)
+		(in_bom yes)
+		(on_board yes)
+		(in_pos_files yes)
+		(dnp no)
+		(property "Reference" "#FLG07"
+			(at 26.67 116.84 0)
+			(show_name no)
+			(do_not_autoplace no)
+			(effects
+				(font
+					(size 1.27 1.27)
+				)
+			)
+		)
+		(property "Value" "PWR_FLAG"
+			(at 26.67 114.3 0)
+			(show_name no)
+			(do_not_autoplace no)
+			(effects
+				(font
+					(size 1.27 1.27)
+				)
+			)
+		)
+		(property "Footprint" ""
+			(at 26.67 110.49 0)
+			(hide yes)
+			(show_name no)
+			(do_not_autoplace no)
+			(effects
+				(font
+					(size 1.27 1.27)
+				)
+			)
+		)
+		(property "Datasheet" ""
+			(at 26.67 110.49 0)
+			(hide yes)
+			(show_name no)
+			(do_not_autoplace no)
+			(effects
+				(font
+					(size 1.27 1.27)
+				)
+			)
+		)
+		(property "Description" "Special symbol for telling ERC where power comes from"
+			(at 26.67 110.49 0)
+			(hide yes)
+			(show_name no)
+			(do_not_autoplace no)
+			(effects
+				(font
+					(size 1.27 1.27)
+				)
+			)
+		)
+		(pin "1"
+		)
+		(instances
+			(project "FE_UFPR_4_0"
+				(path "/0cde0ae3-e31e-4592-8212-8a072a248a80/6442f421-491d-4bfb-bee7-d0b4e843a827"
+					(reference "#FLG07")
+					(unit 1)
+				)
+			)
 		)
 	)
