File: power.kicad_sch (KiCad schematic)
At the start: 70 parts, among them J1 Mini-Fit Jr 5566-02A, Q1 SQD50P06-15L, U1 LMR33630ADDAR, U2 TPS62933FDRLR, U3 AMS1117-3.3, U4 URA2415YMD-6WR3

Commit message: S12.6: JLC feeder fee cut 27 -> 14 Extended codes ($82.89 -> $42.98)
Live re-audit of every Extended line against JLCSearch (2026-09-26); the
2026-09-17 "nothing cuttable" conclusion is partially superseded.

- R10/R11 52.3k/10k -> 68k/13k (both Basic), +5V 4.984 -> 4.985 V
- D1 SMCJ26A -> SMCJ26CA (Preferred, same SMC footprint and grade;
  bidirectional is harmless after Q1), symbol D_TVS, UUID kept
- Vbus R57/R58 2.20k/1.50k -> 3.00k/2.20k (existing RT0603B 0.1% lines):
  VBUS_DIVIDER_RATIO 341.538 -> 327.273, full scale 981.8 V (handoff doc)
- Hand-solder C1, F1-F3, L3, U8, R57/R105, R58/R129, Q1, U5-U7 (HAND=)
- jlc_verify.py --hand-solder: fee counted over codes JLC places
- golden.net re-baselined (field-only diff); ERC 0, DRC 0/0/parity 0,
  fab/ rebuilt (gerbers unchanged)

Co-Authored-By: Claude Opus 5.5 <noreply@anthropic.com>
Parts:
- D1: value SMCJ26A -> SMCJ26CA; symbol FE_UFPR_4_0:D_TVS_Unidirectional -> FE_UFPR_4_0:D_TVS; LCSC C310042 -> C19077605
- R10: value 52.3k -> 68k; LCSC C23198 -> C23231
- R11: value 10k -> 13k; LCSC C25804 -> C22797
Other:
- note added: "S3 - POWER SUPPLIES +24V_IN (18-26V) -> +13V5_GATE 13.500V -> +5V 4.985V -> +3V3 plus isolated +/-15V All component values computed - see S3_POWER_DESIGN.md for every derivation, datasheet equation and JLC stock check."
- note removed: "S3 - POWER SUPPLIES +24V_IN (18-26V) -> +13V5_GATE 13.500V -> +5V 4.984V -> +3V3 plus isolated +/-15V All component values computed - see S3_POWER_DESIGN.md for every derivation, datasheet equation and JLC stock check."
Changed lines of the file:
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@@
 		(comment 3 "See REDESIGN_PLAN.md in project dir")
 	)
-	(text "Q1 REVERSE-POLARITY ORIENTATION (easy to get backwards):\nP-channel body diode conducts DRAIN -> SOURCE, therefore DRAIN = input side, SOURCE = load side.\nNormal polarity: body diode forward + gate pulled to GND by R1 => Vgs approx -24V => hard on.\nReverse polarity: Vgs approx 0 => off, body diode blocks.\nD2 (BZX84C15) IS MANDATORY - unclamped Vgs would be -24..-30V against the +/-20V Vgs limit.\n\nD1 TVS - THE CLAMP MUST STAY BELOW THE BUCK'S ABSOLUTE MAX (this is why it is an SMCJ, not an SMBJ):\nLMR33630 abs max VIN = 38 V. A 600W SMBJ26A clamps to 42.1 V at its rated 14.3 A surge - over the limit.\nSMCJ26A is the 1500W part: same 42.1 V clamp spec but at 35.6 A, so at a realistic surge it sits near\n30-34 V, safely under 38 V. Stand-off 26 V is above the 26 V max rail, so it does not leak in normal use.\nDo NOT substitute an SMBJ here, and do NOT raise the stand-off without re-checking the buck's abs max."
+	(text "Q1 REVERSE-POLARITY ORIENTATION (easy to get backwards):\nP-channel body diode conducts DRAIN -> SOURCE, therefore DRAIN = input side, SOURCE = load side.\nNormal polarity: body diode forward + gate pulled to GND by R1 => Vgs approx -24V => hard on.\nReverse polarity: Vgs approx 0 => off, body diode blocks.\nD2 (BZX84C15) IS MANDATORY - unclamped Vgs would be -24..-30V against the +/-20V Vgs limit.\n\nD1 TVS - THE CLAMP MUST STAY BELOW THE BUCK'S ABSOLUTE MAX (this is why it is an SMCJ, not an SMBJ):\nLMR33630 abs max VIN = 38 V. A 600W SMBJ26A clamps to 42.1 V at its rated 14.3 A surge - over the limit.\nSMCJ26CA (1500W, bidirectional - fine after Q1): same 42.1 V clamp but at 35.7 A, so a realistic surge sits near\n30-34 V, safely under 38 V. Stand-off 26 V is above the 26 V max rail, so it does not leak in normal use.\nDo NOT substitute an SMBJ here, and do NOT raise the stand-off without re-checking the buck's abs max."
 		(exclude_from_sim no)
 		(at 15.24 198 0)
@@
 		)
 	)
-	(text "S3 - POWER SUPPLIES     +24V_IN (18-26V) -> +13V5_GATE 13.500V -> +5V 4.984V -> +3V3    plus isolated +/-15V\nAll component values computed - see S3_POWER_DESIGN.md for every derivation, datasheet equation and JLC stock check."
+	(text "S3 - POWER SUPPLIES     +24V_IN (18-26V) -> +13V5_GATE 13.500V -> +5V 4.985V -> +3V3    plus isolated +/-15V\nAll component values computed - see S3_POWER_DESIGN.md for every derivation, datasheet equation and JLC stock check."
 		(exclude_from_sim no)
 		(at 15.24 16.51 0)
@@
 			)
 		)
-		(property "Value" "52.3k"
+		(property "Value" "68k"
 			(at 304.292 76.835 0)
 			(show_name no)
@@
 			)
 		)
-		(property "LCSC" "C23198"
+		(property "LCSC" "C23231"
 			(at 300.99 74.93 0)
 			(hide yes)
@@
 			)
 		)
-		(property "Value" "10k"
+		(property "Value" "13k"
 			(at 290.322 84.455 0)
 			(show_name no)
@@
 			)
 		)
-		(property "LCSC" "C25804"
+		(property "LCSC" "C22797"
 			(at 287.02 82.55 0)
 			(hide yes)
@@
 	)
 	(symbol
-		(lib_id "FE_UFPR_4_0:D_TVS_Unidirectional")
+		(lib_id "FE_UFPR_4_0:D_TVS")
 		(at 91.44 44.45 270)
 		(unit 1)
@@
 			)
 		)
-		(property "Value" "SMCJ26A"
+		(property "Value" "SMCJ26CA"
 			(at 94.742 46.355 90)
 			(show_name no)
@@
 			)
 		)
-		(property "Description" "Zener diode"
+		(property "Description" "Bidirectional transient-voltage-suppression diode"
 			(at 91.44 44.45 0)
 			(hide yes)
@@
 			)
 		)
-		(property "LCSC" "C310042"
+		(property "LCSC" "C19077605"
 			(at 91.44 44.45 0)
 			(hide yes)
