File: vehicle_io.kicad_sch (KiCad schematic)
At the start: 0 parts

Commit message: S8: vehicle_io sheet, schematic freeze - CAN, isolated cockpit inputs, ECU 5 V feed
vehicle_io: J5 DEUTSCH DTM13-08PA-R004 (8-way, key A - way-count keyed against
the two 12-way keys already used), SN65HVD230 CAN-A front-end with ACT45B
common-mode choke, PSM712 TVS and a bridged-jumper 120 R termination, two
identical optically isolated inputs (LTV-817S high-side, 2.2k pull-down,
SN74LVC2G17 Schmitt - every failure reads LOW), and the provisional +5V_VEH
feed (SS34 back-feed block + 0.2 A polyfuse + SMAJ5.0A). 30 parts, 6 new
symbols, 5 new footprints (DTM13-08PA derived from TE's drawing: it is a
vertical-flange right-angle part with 6.35 mm row spacing, not the flat-base
4.19 mm grid S7's table assumed - corrected there).

Netlist 201/835 -> 220/914, every new net verified node by node; project ERC
--severity-all = 0. golden.net re-baselined. Pin map cross-checked on the
netlist side: 29/29 signals on the SPRUI77 pin the firmware expects. BOM/JLC
audit: 293 placements on 63 LCSC lines (29 Basic / 4 Preferred / 30 Extended),
5 consigned, 0 empty; the 2.2 nF C0G line (C107043, 4 in stock) moved to
Murata C77033 on all ten anti-alias caps.

Tooling: KiCad's vertical-label justify rule was measured and fixed in
layoutlib (every downward GND flag had been drawn over its part on every S7.5
sheet), field justify now follows mirror/180, missing-justify insertion fixed,
and note texts are addressed by content instead of file index. All six older
sheets regenerated: notes identical to HEAD, netlist identical, ERC 0.

Co-Authored-By: Claude Fable 5.1 <noreply@anthropic.com>
Claude-Session: https://claude.ai/code/session_01BbqAgraN6LAYLruGRERKDp
Parts:
- added C116, C118, C119: 100nF 50V, FE_UFPR_4_0:C_0603_1608Metric, symbol FE_UFPR_4_0:C
- added C117: 1uF 50V, FE_UFPR_4_0:C_0805_2012Metric, symbol FE_UFPR_4_0:C
- added D13: PSM712, FE_UFPR_4_0:SOT-23, symbol FE_UFPR_4_0:D_TVS_Dual_CAN
- added D14, D15: 1N4148W, FE_UFPR_4_0:D_SOD-123, symbol FE_UFPR_4_0:D
- added D16: SS34, FE_UFPR_4_0:D_SMA, symbol FE_UFPR_4_0:D_Schottky
- added D17: SMAJ5.0A, FE_UFPR_4_0:D_SMA, symbol FE_UFPR_4_0:D_TVS_Unidirectional
- added F3: 0.2A 30V 1206L020, FE_UFPR_4_0:Fuse_1206_3216Metric, symbol FE_UFPR_4_0:Polyfuse
- added J5: VEH DTM13-08PA-R004 key A, FE_UFPR_4_0:DEUTSCH_DTM13-08PA-R004_Horizontal, symbol FE_UFPR_4_0:Conn_02x04_Counter_Clockwise
- added JP6: CAN TERM bridged=120R, FE_UFPR_4_0:SolderJumper-2_P1.3mm_Bridged_Pad1.0x1.5mm, symbol FE_UFPR_4_0:SolderJumper_2_Bridged
- added L3: ACT45B-101-2P-TL003, FE_UFPR_4_0:L_CommonMode_TDK_ACT45B, symbol FE_UFPR_4_0:L_CommonMode
- added R120, R121: 10k, FE_UFPR_4_0:R_0603_1608Metric, symbol FE_UFPR_4_0:R
- added R122: 120R, FE_UFPR_4_0:R_0603_1608Metric, symbol FE_UFPR_4_0:R
- added R123, R124, R125, R126, R127, R128: 2.2k, FE_UFPR_4_0:R_0603_1608Metric, symbol FE_UFPR_4_0:R
- added TP49: CAN_H, FE_UFPR_4_0:TestPoint_Pad_D1.5mm, symbol FE_UFPR_4_0:TestPoint
- added TP50: CAN_L, FE_UFPR_4_0:TestPoint_Pad_D1.5mm, symbol FE_UFPR_4_0:TestPoint
- added TP51: SW_MAIN_3V3, FE_UFPR_4_0:TestPoint_Pad_D1.5mm, symbol FE_UFPR_4_0:TestPoint
- added TP52: SW_START_3V3, FE_UFPR_4_0:TestPoint_Pad_D1.5mm, symbol FE_UFPR_4_0:TestPoint
- added U18: SN65HVD230DR, FE_UFPR_4_0:SOIC-8_3.9x4.9mm_P1.27mm, symbol FE_UFPR_4_0:SN65HVD230
- added U19, U20: LTV-817S-TA1-C, FE_UFPR_4_0:Optocoupler_LTV-817S_SMD-4P, symbol FE_UFPR_4_0:LTV-817S
- added U21: SN74LVC2G17DBVR, FE_UFPR_4_0:SOT-23-6, symbol FE_UFPR_4_0:74LVC2G17
Connections:
- net CAN_RX_3V3: now also U18.4 (R)
- net CAN_TX_3V3: now also R121.2, U18.1 (D)
- net SW_MAIN_3V3: now also TP51.1, U21.6
- net SW_START_3V3: now also TP52.1, U21.4
- new net: JP6.2 (B), R122.1
- new net: D14.1 (K), R124.2, U19.1
- new net: R125.1, U19.3, U21.1
- new net: D15.1 (K), R127.2, U20.1
- new net: J5.4 (Pin_4), R126.1
- new net: R126.2, R127.1
- new net: D16.1 (K), F3.2
- new net: R123.2, R124.1
- new net: R128.1, U20.3, U21.3
- new net: J5.3 (Pin_3), R123.1
- new net +3V3: C116.1, C117.1, C118.1, R121.1, U18.3 (VCC), U19.4, U20.4, U21.5 (VCC)
- new net +5V: D16.2 (A)
- new net +5V_VEH: C119.1, D17.1 (K), F3.1, J5.2 (Pin_2)
- new net CAN_H: D13.1 (K), J5.1 (Pin_1), L3.1, R122.2, TP49.1
- new net CAN_H_XCVR: L3.4, U18.7 (CANH)
- new net CAN_L: D13.2 (K), J5.8 (Pin_8), JP6.1 (A), L3.2, TP50.1
- new net CAN_L_XCVR: L3.3, U18.6 (CANL)
- new net CAN_RS: R120.1, U18.8 (Rs)
- new net GND: C116.2, C117.2, C118.2, C119.2, D13.3 (A), D17.2 (A), J5.7 (Pin_7), R120.2, R125.2, R128.2, U18.2 (GND), U21.2 (GND)
- new net SW_MAIN_RTN: D14.2 (A), J5.6 (Pin_6), U19.2
- new net SW_START_RTN: D15.2 (A), J5.5 (Pin_5), U20.2
- no-connect marks 0 -> 1
Other:
- note added: "+5V_VEH (PROVISIONAL, user confirming with the ECU team): if the ECU's isolated transceiver powers its bus side from us, this is the pin. F3 0.2 A polyfuse (trips 0.46 A) + D16 SS34 + D17 SMAJ5.0A + C119. D16 blocks anything on the harness from back-feeding our +5V rail (the polyfuse alone would let a mis-wired 12 V reach every 5 V part on the board); the price is ~0.25 V: expect 4.6..4.75 V at <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"
- note added: "CAN (S8): CAN-A, GPIO4 TX / GPIO5 RX = LaunchPad J4-36 / J4-35, on J21. U18 SN65HVD230 (3.3 V, JLC Preferred). This is a dedicated 2-node link to the ECU; the galvanic barrier is on the ECU side (ISO1042/ISO1050 or ISOW1044), so OUR node is the non-isolated reference its bus side follows. Termination: 2 nodes => both ends terminated => R122 120R is FITTED by default through the bridged jumper JP6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"
- note added: "ISOLATED COCKPIT INPUTS (S8): identical channels, drawn identically. Input accepts 8..30 V DC (nominal 12 V GLV, the AM06 ECU runs on +12V) referenced to its own RTN pin = car GND. Our logic 24 V is a separate battery unbonded from the car, so every car-referenced signal crosses an optocoupler (LTV-817S-C, 5 kV, JLC Basic, CTR 200..400 %). LED chain 2 x 2.2k = 4.4k: 1.5 mA @ 8 V, 2.5 mA @ 12 V, 5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"
- note added: "J5 - VEHICLE CONNECTOR: DEUTSCH DTM13-08PA-R004, 8-way, key A (CONSIGNED) cav 1 CAN_H cav 8 CAN_L (twisted pair, adjacent cavities) cav 2 +5V_VEH out cav 7 GND (ECU isolated-side supply, PROVISIONAL) cav 3 SW_MAIN_IN cav 6 SW_MAIN_RTN (FSAE shutdown circuit, car-referenced) cav 4 SW_START_IN cav 5 SW_START_RTN (start button, car-referenced) Every function sits on a physically adjacent pair (1-8, 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"
- note added: "S9 LAYOUT RULES FOR THIS SHEET 1. J5 on the service edge next to the 24 V entry; board edge on the footprint's Dwgs.User line; flange bracket - see the J5 note. 2. CAN pair: keep CAN_H/CAN_L routed as a pair from U18 to J5, D13 and the termination right at the connector, L3 between them and U18. 3. The opto LED side (J5 cav 3-6, R123/R124/R126/R127, D14/D15) is CAR- referenced: no GND pour under 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"
