File: vehicle_io.kicad_sch (KiCad schematic)
At the start: 30 parts, among them J5 VEH DTM13-08PA-R004 key A, U18 SN65HVD230DR, U19 LTV-817S-TA1-C, U20 LTV-817S-TA1-C, U21 SN74LVC2G17DBVR

Commit message: POwer interface fixes
Changed lines of the file:
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@@
 		)
+	)
+	(junction
+		(at 91.44 38.1)
+		(diameter 0)
+		(color 0 0 0 0)
+	)
+	(junction
+		(at 68.58 38.1)
+		(diameter 0)
+		(color 0 0 0 0)
 	)
 	(no_connect
@@
 	(wire
 		(pts
+			(xy 50.8 71.12) (xy 58.42 71.12)
+		)
+		(stroke
+			(width 0)
+			(type default)
+		)
+	)
+	(wire
+		(pts
 			(xy 58.42 71.12) (xy 58.42 38.1)
 		)
@@
 		)
 		(stroke
-			(width 0)
-			(type default)
-		)
-	)
-	(wire
-		(pts
-			(xy 50.8 71.12) (xy 58.42 71.12)
-		)
-		(stroke
