File: vehicle_io.kicad_sch (KiCad schematic)
At the start: 30 parts, among them J5 VEH DTM13-08PA-R004 key A, U18 SN65HVD230DR, U19 LTV-817S-TA1-C, U20 LTV-817S-TA1-C, U21 SN74LVC2G17DBVR

Commit message: S12.5: J3/J4/J5 swapped to vertical DEUTSCH DT15 headers (TE sample-program constraint)
- DT15-12PA (J3, key A), DT15-12PB (J4, key B), DT15-08PD (J5, key D); symbols/netlist unchanged
- new footprints DEUTSCH_DT15-12P_Vertical / DEUTSCH_DT15-08P_Vertical + STEP bodies (gen_3d_dt15.py),
  hand-derived from TE drawings C-DT15-12PX rev D2 / C-DT15-08PX-XXXX rev A (datasheets/)
- board: footprint blocks swapped on a scratch copy and spliced; NOT re-placed/re-routed yet (DRC 653 at old positions)
- golden.net re-baselined (S12's C22935 fix), J5 MPN/Manufacturer added, sheet notes rewritten
- docs: CLAUDE.md phase, DECISION_LOG, OPEN_ITEMS, LIBRARY, JLC_PARTS, VERIFIED_FACTS, TOOLING_NOTES, S9_6, fab/README stale banner

Co-Authored-By: Claude Fable 5.1 <noreply@anthropic.com>
Parts:
- J5: value VEH DTM13-08PA-R004 key A -> VEH DT15-08PD key D; footprint FE_UFPR_4_0:DEUTSCH_DTM13-08PA-R004_Horizontal -> FE_UFPR_4_0:DEUTSCH_DT15-08P_Vertical; MPN (none) -> DT15-08PD; Manufacturer (none) -> TE Connectivity / DEUTSCH
Other:
- note added: "J5 - VEHICLE CONNECTOR: DEUTSCH DT15-08PD, 8-way VERTICAL (180 deg) flanged receptacle, key D (TE student-sample program, 2026-09-23) cav 1 CAN_H cav 8 CAN_L (twisted pair, adjacent cavities) cav 2 +5V_VEH out cav 7 GND (ECU isolated-side supply, PROVISIONAL) cav 3 SW_MAIN_IN cav 6 SW_MAIN_RTN (FSAE shutdown circuit, car-referenced) cav 4 SW_START_IN cav 5 SW_START_RTN (start button, car-referenc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"
- note removed: "J5 - VEHICLE CONNECTOR: DEUTSCH DTM13-08PA-R004, 8-way, key A (CONSIGNED) cav 1 CAN_H cav 8 CAN_L (twisted pair, adjacent cavities) cav 2 +5V_VEH out cav 7 GND (ECU isolated-side supply, PROVISIONAL) cav 3 SW_MAIN_IN cav 6 SW_MAIN_RTN (FSAE shutdown circuit, car-referenced) cav 4 SW_START_IN cav 5 SW_START_RTN (start button, car-referenced) Every function sits on a physically adjacent pair (1-8, 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"
Changed lines of the file:
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@@
 		)
 	)
-	(text "J5 - VEHICLE CONNECTOR: DEUTSCH DTM13-08PA-R004, 8-way, key A (CONSIGNED)\ncav 1  CAN_H          cav 8  CAN_L         (twisted pair, adjacent cavities)\ncav 2  +5V_VEH out    cav 7  GND           (ECU isolated-side supply, PROVISIONAL)\ncav 3  SW_MAIN_IN     cav 6  SW_MAIN_RTN   (FSAE shutdown circuit, car-referenced)\ncav 4  SW_START_IN    cav 5  SW_START_RTN  (start button, car-referenced)\nEvery function sits on a physically adjacent pair (1-8, 2-7, 3-6, 4-5).\nWHY 8-WAY: the two DTM13-12P-R005 on this board use keys A and B, and TE's\nboard-mount DTM13 family exists only in 8- and 12-way. A 12-way plug cannot\nenter this 8-way receptacle, so mis-mating the LEM or encoder harness into the\nvehicle socket (or vice versa) is impossible by way-count.\n!! -R004 is a VERTICAL PANEL FLANGE (68.58 x 33.02 + 4 ears, slots 8.89 x 2.54),\nnot a flat base like the 12-way -R005: flange + housing hang beyond the board\nedge and the flange reaches 4.4 mm below the board. Only the 8 pins hold it.\nS9 must (a) put the board edge on the footprint's Dwgs.User line and (b) add a\nbracket or panel to the flange slots. Cavity numbers taken from the 8-way\ndrawing (which labels them): near row 1-4, far row 5-8 - confirm on a real\nDTM06-08SA before crimping, like J3/J4."
+	(text "J5 - VEHICLE CONNECTOR: DEUTSCH DT15-08PD, 8-way VERTICAL (180 deg) flanged receptacle, key D  (TE student-sample program, 2026-09-23)\ncav 1  CAN_H          cav 8  CAN_L         (twisted pair, adjacent cavities)\ncav 2  +5V_VEH out    cav 7  GND           (ECU isolated-side supply, PROVISIONAL)\ncav 3  SW_MAIN_IN     cav 6  SW_MAIN_RTN   (FSAE shutdown circuit, car-referenced)\ncav 4  SW_START_IN    cav 5  SW_START_RTN  (start button, car-referenced)\nEvery function sits on a physically adjacent pair (1-8, 2-7, 3-6, 4-5).\nSwapped 2026-09-23 from the right-angle DTM13-08PA-R004 (whose panel flange hung past the board edge).\nWHY 8-WAY / KEY D: J3 and J4 are 12-way keys A/B; a 12-way plug cannot enter this 8-way receptacle,\nand key D also excludes every key-A/B/C 8-way plug. DT15-08PD is the only vertical 8-way header in\nTE's sample program; its plug DT06-08SD is NOT sampleable (DT06-08SA, key A, is) - settle the plug\nsource before crimping. Plug + W8S wedgelock, size-16 contacts 0462-201-16141 / 1062-16-0122.\nPin numbers = cavity numbers on TE drawing C-DT15-08PX sheets 1-2 (mating face: pin 1 bottom-left,\n1-4 up the left column, 5-8 down the right). Recommended PCB layout is printed on sheet 2.\nBoard side: 35.26 x 55.12 body on the board, flange 15.5 mm up, 4x #4-20 Plastite screws from the\nboard UNDERSIDE (heads on B.Cu - keep copper clear of the B.CrtYd circles)."
 		(exclude_from_sim no)
 		(at 220.98 20.32 0)
@@
 			)
 		)
-		(property "Value" "VEH DTM13-08PA-R004 key A"
+		(property "Value" "VEH DT15-08PD key D"
 			(at 36.83 87.63 0)
 			(show_name no)
@@
 			)
 		)
-		(property "Footprint" "FE_UFPR_4_0:DEUTSCH_DTM13-08PA-R004_Horizontal"
+		(property "Footprint" "FE_UFPR_4_0:DEUTSCH_DT15-08P_Vertical"
 			(at 45.72 73.66 0)
 			(hide yes)
@@
 			(at 45.72 73.66 0)
 			(hide yes)
+			(show_name no)
+			(do_not_autoplace no)
+			(effects
+				(font
+					(size 1.27 1.27)
+				)
+			)
+		)
+		(property "MPN" "DT15-08PD"
+			(at 45.72 73.66 0)
+			(hide yes)
+			(show_name no)
+			(do_not_autoplace no)
+			(effects
+				(font
+					(size 1.27 1.27)
+				)
+			)
+		)
+		(property "Manufacturer" "TE Connectivity / DEUTSCH"
+			(at 45.72 73.66 0)
+			(hide yes)
