File: FE_UFPR_4_0.kicad_pcb (KiCad board)
At the start: 4 copper layers, 146 x 130 mm, 368 parts, among them J1 Mini-Fit Jr 5566-02A, J2 DSUB-37_Socket, J20 LaunchPad J1+J3, J21 LaunchPad J4+J2, J22 LaunchPad J5+J7, J23 LaunchPad J8+J6, J3 LEM DTM13-12PA-R005 key A, J4 ENC DTM13-12PB-R005 key B, J5 VEH DTM13-08PA-R004 key A, Q1 SQD50P06-15L, U1 LMR33630ADDAR, U10 SN74LVC2G17DBVR, U11 SN74LVC2G17DBVR, U12 OPA2376, U13 OPA2376, U14 OPA2376, U15 OPA2376, U16 OPA2376, U17 OPA2376, U18 SN65HVD230DR, U19 LTV-817S-TA1-C, U2 TPS62933FDRLR, U20 LTV-817S-TA1-C, U21 SN74LVC2G17DBVR, U3 AMS1117-3.3, U4 URA2415YMD-6WR3, U5 UCC27524DR, U6 UCC27524DR, U7 UCC27524DR, U8 SN74LVC1G11DBVR, U9 SN74LVC2G17DBVR

Commit message: fixing drc warnings
Parts:
- added LOGO1: Logo_UFPR_Formula_32mm, FE_UFPR_4_0:Logo_UFPR_Formula_32mm, F.Cu at (178.7, 122.3)
Routing:
- net /gate_drive/MOD_AUX15V_1: track 47.2 -> 59.4 mm
- net /gate_drive/MOD_AUX15V_2: track 43.4 -> 55.5 mm
- net /current_sense/ISNS_VREF: track 120.8 -> 122.6 mm
- net /encoder/ENC_VREF3V: track 19.0 -> 20.9 mm
- net /power/PWR_LED_5V: track 0.00 -> 1.85 mm
- net /gate_drive/SHIELD_DB37: track 89.9 -> 88.7 mm

Commit message: Logos on silk
Parts:
- removed LOGO1: Logo_UFPR_Formula_32mm, FE_UFPR_4_0:Logo_UFPR_Formula_32mm
- added LOGO**: Logo_UFPR_Formula_16mm, FE_UFPR_4_0:Logo_UFPR_Formula_16mm, F.Cu at (263.0, 179.6)
- added LOGO**: Logo_UFPR_Formula_32mm, FE_UFPR_4_0:Logo_UFPR_Formula_32mm, B.Cu at (140.8, 110.6)
Routing:
- net GND: track 46.3 -> 271.4 mm, vias 72 -> 402
- net /gate_drive/PWM_UH_15V: track 70.9 -> 70.0 mm
- net +3V3: vias 22 -> 24
- net (no net): vias 6 -> 0
