File: _restore_backup_2026-09-17T15-06-19-842/FE_UFPR_4_0.kicad_pcb (KiCad board)
At the start: 4 copper layers, 146.1 x 130 mm, 374 parts, among them J1 Mini-Fit Jr 5566-02A, J2 DSUB-37_Socket, J20 LaunchPad J1+J3, J21 LaunchPad J4+J2, J22 LaunchPad J5+J7, J23 LaunchPad J8+J6, J3 LEM DTM13-12PA-R005 key A, J4 ENC DTM13-12PB-R005 key B, J5 VEH DTM13-08PA-R004 key A, Q1 SQD50P06-15L, U1 LMR33630ADDAR, U10 SN74LVC2G17DBVR, U11 SN74LVC2G17DBVR, U12 OPA2376, U13 OPA2376, U14 OPA2376, U15 OPA2376, U16 OPA2376, U17 OPA2376, U18 SN65HVD230DR, U19 LTV-817S-TA1-C, U2 TPS62933FDRLR, U20 LTV-817S-TA1-C, U21 SN74LVC2G17DBVR, U3 AMS1117-3.3, U4 URA2415YMD-6WR3, U5 UCC27524DR, U6 UCC27524DR, U7 UCC27524DR, U8 SN74LVC1G11DBVR, U9 SN74LVC2G17DBVR

Commit message: Placing
Parts:
- moved TP22 253.5 mm to (312.4, 201.6)
- moved TP19 252.1 mm to (306.9, 198.5)
- moved TP21 252.0 mm to (310.0, 198.5)
- moved TP47 217.4 mm to (299.1, 153.4)
- moved R62 137.0 mm to (200.5, 109.7)
- moved C59 137.0 mm to (200.7, 115.6)
- moved C61 137.0 mm to (204.3, 109.9)
- moved R59 137.0 mm to (203.6, 112.2)
- moved TP20 137.0 mm to (204.2, 115.9)
- moved TP23 137.0 mm to (200.2, 112.8)
- moved D12 114.2 mm to (297.7, 144.8), turned to 180 degrees
- moved C115 104.9 mm to (300.9, 139.2), turned to 0 degrees
- moved C114 102.7 mm to (296.9, 137.6), turned to 0 degrees
- moved C10 59.7 mm to (268.3, 137.0)
- moved C11 59.7 mm to (262.8, 136.7)
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Other:
- board size 146.1 x 130 mm -> 159.6 x 130 mm
