File: _restore_backup_2026-09-22T22-07-53-839/FE_UFPR_4_0.kicad_pcb (KiCad board)
At the start: 4 copper layers, 146 x 130 mm, 370 parts, among them J1 Mini-Fit Jr 5566-02A, J2 DSUB-37_Socket, J20 LaunchPad J1+J3, J21 LaunchPad J4+J2, J22 LaunchPad J5+J7, J23 LaunchPad J8+J6, J3 LEM DTM13-12PA-R005 key A, J4 ENC DTM13-12PB-R005 key B, J5 VEH DTM13-08PA-R004 key A, Q1 SQD50P06-15L, U1 LMR33630ADDAR, U10 SN74LVC2G17DBVR, U11 SN74LVC2G17DBVR, U12 OPA2376, U13 OPA2376, U14 OPA2376, U15 OPA2376, U16 OPA2376, U17 OPA2376, U18 SN65HVD230DR, U19 LTV-817S-TA1-C, U2 TPS62933FDRLR, U20 LTV-817S-TA1-C, U21 SN74LVC2G17DBVR, U3 AMS1117-3.3, U4 URA2415YMD-6WR3, U5 UCC27524DR, U6 UCC27524DR, U7 UCC27524DR, U8 SN74LVC1G11DBVR, U9 SN74LVC2G17DBVR

Commit message: more routing
Parts:
- moved TP17 77.2 mm to (261.1, 211.5)
- moved TP18 75.0 mm to (261.1, 207.3)
- moved TP14 41.3 mm to (262.1, 231.9)
- moved TP12 40.7 mm to (267.4, 231.9)
- moved TP10 40.7 mm to (272.9, 231.9)
- moved TP15 37.2 mm to (259.4, 231.9)
- moved TP13 37.1 mm to (264.8, 231.9)
- moved TP11 36.9 mm to (270.1, 231.9)
- moved FB1 35.5 mm to (209.8, 102.9), turned to -90 degrees
- moved C111 27.7 mm to (208.9, 107.9)
- moved C112 27.7 mm to (208.8, 105.9)
- moved R120 14.4 mm to (227.7, 119.2), turned to 0 degrees
- moved TP5 9.67 mm to (252.0, 207.2)
- moved U18 8.14 mm to (229.3, 115.5), turned to 180 degrees
- moved R132 5.87 mm to (203.9, 112.3), turned to 0 degrees
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Connections:
- J22 pad 12: /ISNS_C_ADC -> /ISNS_A_ADC
- J22 pad 16: /ISNS_A_ADC -> /ISNS_C_ADC
- U4 pad 2: +24V_MOD -> +24V_PROT
Routing:
- net /NTC_1_ADC: track 100.7 -> 0.00 mm, vias 2 -> 0
- net /VBUS_ADC: track 91.6 -> 0.00 mm, vias 4 -> 0
- net /ISNS_A_RAW: track 90.0 -> 0.00 mm
- net /ISNS_B_RAW: track 70.4 -> 0.00 mm
- net +15V_ISO: track 83.3 -> 24.3 mm
- net /encoder/ENC_VDD: track 86.0 -> 30.7 mm, vias 3 -> 0
- net -15V_ISO: track 70.5 -> 21.3 mm
- net /ISNS_C_RAW: track 47.5 -> 0.00 mm, vias 2 -> 0
- net /gate_drive/MOD_AUX15V_1: track 43.9 -> 0.00 mm, vias 1 -> 0
- net /gate_drive/MOD_AUX15V_2: track 40.2 -> 0.00 mm, vias 1 -> 0
- net /encoder/MOT_TEMP_RAW: track 81.3 -> 41.3 mm, vias 2 -> 0
- net +3V3: track 36.4 -> 16.0 mm, vias 2 -> 0
- net /encoder/ENC_VREF_HI: track 21.4 -> 1.27 mm, vias 2 -> 0
- net /ENC_SIN_ADC: track 34.0 -> 14.3 mm
- net /SW_START_3V3: track 15.6 -> 0.00 mm
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- removed copper zone on B.Cu, net +13V5_GATE
- removed copper zone on F.Cu, net +3V3
- removed copper zone on B.Cu, net +5V
- removed copper zone on B.Cu, net GND
