File: _restore_backup_2026-09-22T22-07-53-839/power.kicad_sch (KiCad schematic)
At the start: 70 parts, among them J1 Mini-Fit Jr 5566-02A, Q1 SQD50P06-15L, U1 LMR33630ADDAR, U2 TPS62933FDRLR, U3 AMS1117-3.3, U4 URA2415YMD-6WR3

Commit message: more routing
Connections:
- net +24V_MOD: no longer U4.2 (+Vin)
- net +24V_PROT: now also U4.2 (+Vin)
Changed lines of the file:
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@@
 		)
 	)
-	(global_label "+24V_MOD"
+	(global_label "+24V_PROT"
 		(shape bidirectional)
 		(at 219.71 125.73 180)
